File: board/weit_generator/filter.kicad_sch (KiCad schematic)
At the start: 10 parts

Commit message: .
Parts:
- removed U? (x2): MCP6004, Package_SO:SOIC-14_3.9x8.7mm_P1.27mm, symbol Amplifier_Operational:MCP6004
- added U1: MCP6004, Package_DIP:DIP-14_W7.62mm_Socket_LongPads, symbol Amplifier_Operational:MCP6004
Connections:
- net OUT: now also U1.8, U1.9 (-)
- net at C?.2, R?.2: now also U1.10 (+)
- net at C?.1, C?.1, R?.2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: now also U1.5 (+)
- net at R?.1: now also U1.6 (-), U1.7
