File: board/weit_generator/_autosave-weit_generator.kicad_pcb (KiCad board)
At the start: 2 copper layers, 58 parts, among them J1 POWER, J2 PROG, J3 OUTPUT, Q1 BC547, U1 MCP6004, U2 AVR32DA28x-xSO, U3 LM4041L, U4 LMV321, X1 SG-5032CAN

Commit message: New layout
Parts:
- moved J2 77.2 mm to (123.5, 88.0), turned to 180 degrees
- moved C1 59.6 mm to (154.7, 87.0), turned to 180 degrees
- moved Q1 19.4 mm to (116.4, 130.4), turned to 0 degrees
- moved R2 18.0 mm to (126.6, 104.7), turned to -90 degrees
- moved R29 17.7 mm to (112.9, 125.0)
- moved J1 17.3 mm to (154.8, 93.0), turned to -90 degrees
- moved RV1 17.1 mm to (123.4, 117.6), turned to 90 degrees
- moved TP3 14.7 mm to (149.1, 127.0)
- moved C2 14.1 mm to (117.8, 122.7), turned to 90 degrees
- moved R27 13.3 mm to (122.1, 125.7), turned to 0 degrees
- moved R28 13.0 mm to (118.7, 125.7), turned to 180 degrees
- moved TP2 12.5 mm to (111.7, 140.2)
- moved R21 11.8 mm to (139.6, 97.7), turned to 180 degrees
- moved C6 11.5 mm to (166.2, 117.5), turned to -90 degrees
- moved C13 9.42 mm to (124.6, 129.4), turned to -90 degrees
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Routing:
- net +3V0: track 33.2 -> 163.1 mm
- net GND: track 11.6 -> 27.8 mm
- net Net-(U1C--): track 38.2 -> 24.2 mm
- net /Autogain/OUT: track 4.72 -> 17.5 mm
- net Net-(J2-Pin_2): track 5.18 -> 12.8 mm
- net Net-(U1C-+): track 13.5 -> 20.8 mm
- net Net-(C13-Pad1): track 26.1 -> 19.3 mm
- net Net-(C11-Pad2): track 21.5 -> 15.5 mm
- net /Output Filter/IN: track 41.5 -> 36.6 mm
- net /R-2R DAC/OUT: track 3.57 -> 8.29 mm
- net Net-(J2-Pin_3): track 7.83 -> 11.3 mm
- net /Autogain/IN: track 27.9 -> 24.5 mm
- net Net-(D2-K): track 3.44 -> 6.70 mm
- net Net-(U1A--): track 9.35 -> 6.21 mm
- net Net-(U1D-+): track 12.7 -> 9.83 mm
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- added copper zone on F.Cu, net GND
Other:
- board outline added: 75 x 64.6 mm
