File: board/weit_generator/weit_generator.kicad_sch (KiCad schematic)
At the start: 19 parts, among them J1 POWER, J2 PROG, J3 OUTPUT, U1 MCP6004, U2 AVR32DA28x-xSO, X1 SG-5032CAN

Commit message: .
Parts:
- renumbered C6 to C1, C2 to C10, C1 to C2, C7 to C4, C4 to C5, C5 to C6, R2 to R15, R3 to R20, R1 to R23, U2 to U1, U1 to U2
Changed lines of the file:
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@@
   (symbol (lib_id "Amplifier_Operational:MCP6004") (at 48.26 128.905 0) (unit 2)
     (in_bom yes) (on_board yes) (dnp no) (fields_autoplaced)
-    (property "Reference" "U1" (at 48.26 120.015 0)
+    (property "Reference" "U2" (at 48.26 120.015 0)
       (effects (font (size 1.27 1.27)))
     )
@@
       (project "weit_generator"
         (path "/b85c55a9-e1f6-4dbf-a795-73634abf8d52"
-          (reference "U1") (unit 2)
+          (reference "U2") (unit 2)
         )
         (path "/b85c55a9-e1f6-4dbf-a795-73634abf8d52/97b440c2-49e0-43c1-8dbd-070a3fa32fe0"
@@
   (symbol (lib_id "Device:C_Polarized") (at 110.49 163.195 0) (unit 1)
     (in_bom yes) (on_board yes) (dnp no) (fields_autoplaced)
-    (property "Reference" "C1" (at 114.3 161.671 0)
+    (property "Reference" "C2" (at 114.3 161.671 0)
       (effects (font (size 1.27 1.27)) (justify left))
     )
@@
       (project "weit_generator"
         (path "/b85c55a9-e1f6-4dbf-a795-73634abf8d52"
-          (reference "C1") (unit 1)
+          (reference "C2") (unit 1)
         )
       )
@@
   (symbol (lib_id "MCU_Microchip_AVR_Dx:AVR32DA28x-xSO") (at 83.82 64.77 0) (mirror y) (unit 1)
     (in_bom yes) (on_board yes) (dnp no)
-    (property "Reference" "U2" (at 81.8641 90.805 0)
+    (property "Reference" "U1" (at 81.8641 90.805 0)
       (effects (font (size 1.27 1.27)) (justify left))
     )
@@
       (project "weit_generator"
         (path "/b85c55a9-e1f6-4dbf-a795-73634abf8d52"
-          (reference "U2") (unit 1)
+          (reference "U1") (unit 1)
         )
       )
@@
   (symbol (lib_id "Device:C") (at 144.78 163.83 0) (unit 1)
     (in_bom yes) (on_board yes) (dnp no) (fields_autoplaced)
-    (property "Reference" "C5" (at 148.59 163.195 0)
+    (property "Reference" "C6" (at 148.59 163.195 0)
       (effects (font (size 1.27 1.27)) (justify left))
     )
@@
       (project "weit_generator"
         (path "/b85c55a9-e1f6-4dbf-a795-73634abf8d52"
-          (reference "C5") (unit 1)
+          (reference "C6") (unit 1)
         )
       )
@@
   (symbol (lib_id "Device:C") (at 231.14 76.835 90) (mirror x) (unit 1)
     (in_bom yes) (on_board yes) (dnp no)
-    (property "Reference" "C7" (at 231.14 82.55 90)
+    (property "Reference" "C4" (at 231.14 82.55 90)
       (effects (font (size 1.27 1.27)))
     )
@@
       (project "weit_generator"
         (path "/b85c55a9-e1f6-4dbf-a795-73634abf8d52"
-          (reference "C7") (unit 1)
+          (reference "C4") (unit 1)
         )
       )
@@
   (symbol (lib_id "Amplifier_Operational:MCP6004") (at 90.17 165.1 0) (unit 5)
     (in_bom yes) (on_board yes) (dnp no) (fields_autoplaced)
-    (property "Reference" "U1" (at 88.9 164.465 0)
+    (property "Reference" "U2" (at 88.9 164.465 0)
       (effects (font (size 1.27 1.27)) (justify left))
     )
@@
       (project "weit_generator"
         (path "/b85c55a9-e1f6-4dbf-a795-73634abf8d52"
-          (reference "U1") (unit 5)
+          (reference "U2") (unit 5)
         )
       )
@@
   (symbol (lib_id "Device:C") (at 231.14 69.85 90) (unit 1)
     (in_bom yes) (on_board yes) (dnp no) (fields_autoplaced)
-    (property "Reference" "C6" (at 231.14 64.135 90)
+    (property "Reference" "C1" (at 231.14 64.135 90)
       (effects (font (size 1.27 1.27)))
     )
@@
       (project "weit_generator"
         (path "/b85c55a9-e1f6-4dbf-a795-73634abf8d52"
-          (reference "C6") (unit 1)
+          (reference "C1") (unit 1)
         )
       )
@@
   (symbol (lib_id "Device:C") (at 107.315 132.715 0) (unit 1)
     (in_bom yes) (on_board yes) (dnp no) (fields_autoplaced)
-    (property "Reference" "C2" (at 111.125 132.08 0)
+    (property "Reference" "C10" (at 111.125 132.08 0)
       (effects (font (size 1.27 1.27)) (justify left))
     )
@@
       (project "weit_generator"
         (path "/b85c55a9-e1f6-4dbf-a795-73634abf8d52"
-          (reference "C2") (unit 1)
+          (reference "C10") (unit 1)
         )
       )
@@
   (symbol (lib_id "Device:R") (at 89.535 128.905 90) (unit 1)
     (in_bom yes) (on_board yes) (dnp no) (fields_autoplaced)
-    (property "Reference" "R1" (at 89.535 123.825 90)
+    (property "Reference" "R23" (at 89.535 123.825 90)
       (effects (font (size 1.27 1.27)))
     )
@@
       (project "weit_generator"
         (path "/b85c55a9-e1f6-4dbf-a795-73634abf8d52"
-          (reference "R1") (unit 1)
+          (reference "R23") (unit 1)
         )
         (path "/b85c55a9-e1f6-4dbf-a795-73634abf8d52/97b440c2-49e0-43c1-8dbd-070a3fa32fe0"
@@
   (symbol (lib_id "Device:C") (at 133.35 163.83 0) (unit 1)
     (in_bom yes) (on_board yes) (dnp no) (fields_autoplaced)
-    (property "Reference" "C4" (at 137.16 163.195 0)
+    (property "Reference" "C5" (at 137.16 163.195 0)
       (effects (font (size 1.27 1.27)) (justify left))
     )
@@
       (project "weit_generator"
         (path "/b85c55a9-e1f6-4dbf-a795-73634abf8d52"
-          (reference "C4") (unit 1)
+          (reference "C5") (unit 1)
         )
       )
@@
   (symbol (lib_id "Device:R_Photo") (at 153.035 78.105 180) (unit 1)
     (in_bom yes) (on_board yes) (dnp no)
-    (property "Reference" "R3" (at 145.415 77.47 0)
+    (property "Reference" "R20" (at 145.415 77.47 0)
       (effects (font (size 1.27 1.27)) (justify right))
     )
@@
       (project "weit_generator"
         (path "/b85c55a9-e1f6-4dbf-a795-73634abf8d52"
-          (reference "R3") (unit 1)
+          (reference "R20") (unit 1)
         )
       )
@@
   (symbol (lib_id "Device:R") (at 147.32 71.12 270) (mirror x) (unit 1)
     (in_bom yes) (on_board yes) (dnp no)
-    (property "Reference" "R2" (at 147.32 66.675 90)
+    (property "Reference" "R15" (at 147.32 66.675 90)
       (effects (font (size 1.27 1.27)))
     )
@@
       (project "weit_generator"
         (path "/b85c55a9-e1f6-4dbf-a795-73634abf8d52"
-          (reference "R2") (unit 1)
-        )
-      )
+          (reference "R15") (unit 1)
+        )
+      )

Commit message: .
Other:
- moved on the sheet: C1, C4, J1, J3, U2B

Commit message: WIELKA POLONIAAAAA
Parts:
- J1: value POWER -> Zasilanie
- J3: value OUTPUT -> Wyjście
Other:
- sheet Autogain renamed Kontrola Amplitiudy
- sheet Output Filter renamed Filtr Wyjściowy
- note added: "Rezystor kontrolowany prądowo. Tłumi sygnał"
- note removed: "Crude voltage-controlled-resistor, works as an attenuator"
- title: (none) -> Generator 1kHz
- moved on the sheet: C2
Changed lines of the file:
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@@
 (kicad_sch (version 20230121) (generator eeschema)
   (paper "A4")
+  (title_block
+    (title "Generator 1kHz")
+    (date "2023-04-15")
+    (rev "1.0")
+    (comment 1 "Kondensatory C1, C1 polipropylenowe")
+    (comment 2 "Częstotliwość X1 12,288Mhz")
+  )
   (junction (at 153.035 71.12) (diameter 0) (color 0 0 0 0)
   )
@@
     (stroke (width 0) (type default))
   )
+  (wire (pts (xy 68.58 160.655) (xy 68.58 164.465))
+    (stroke (width 0) (type default))
+  )
   (wire (pts (xy 211.455 71.12) (xy 211.455 75.565))
     (stroke (width 0) (type default))
@@
     (stroke (width 0) (type default))
   )
+  (wire (pts (xy 68.58 170.18) (xy 68.58 167.005))
+    (stroke (width 0) (type default))
+  )
   (wire (pts (xy 133.985 71.12) (xy 136.525 71.12))
     (stroke (width 0) (type default))
@@
     (fill (type none))
   )
-  (text "Crude voltage-controlled-resistor, works as an attenuator"
-    (at 111.125 94.615 0)
+  (text "Rezystor kontrolowany prądowo. Tłumi sygnał" (at 137.16 92.71 0)
     (effects (font (size 1 1)) (justify left bottom))
   )
@@
     )
   )
-  (symbol (lib_id "power:+3V0") (at 68.58 164.465 0) (mirror y) (unit 1)
+  (symbol (lib_id "power:+3V0") (at 68.58 160.655 0) (mirror y) (unit 1)
     (in_bom yes) (on_board yes) (dnp no)
-    (property "Reference" "#PWR03" (at 68.58 168.275 0)
-      (effects (font (size 1.27 1.27)) hide)
-    )
-    (property "Value" "+3V0" (at 68.58 160.655 0)
-      (effects (font (size 1.27 1.27)))
-    )
-    (property "Footprint" "" (at 68.58 164.465 0)
-      (effects (font (size 1.27 1.27)) hide)
-    )
-    (property "Datasheet" "" (at 68.58 164.465 0)
+    (property "Reference" "#PWR03" (at 68.58 164.465 0)
+      (effects (font (size 1.27 1.27)) hide)
+    )
+    (property "Value" "+3V0" (at 68.58 156.845 0)
+      (effects (font (size 1.27 1.27)))
+    )
+    (property "Footprint" "" (at 68.58 160.655 0)
+      (effects (font (size 1.27 1.27)) hide)
+    )
+    (property "Datasheet" "" (at 68.58 160.655 0)
       (effects (font (size 1.27 1.27)) hide)
     )
@@
     )
   )
-  (symbol (lib_id "Device:C_Polarized") (at 110.49 163.195 0) (unit 1)
-    (in_bom yes) (on_board yes) (dnp no) (fields_autoplaced)
-    (property "Reference" "C2" (at 114.3 161.671 0)
-      (effects (font (size 1.27 1.27)) (justify left))
-    )
-    (property "Value" "100u" (at 114.3 164.211 0)
-      (effects (font (size 1.27 1.27)) (justify left))
-    )
-    (property "Footprint" "Capacitor_THT:CP_Radial_D6.3mm_P2.50mm" (at 111.4552 167.005 0)
-      (effects (font (size 1.27 1.27)) hide)
-    )
-    (property "Datasheet" "~" (at 110.49 163.195 0)
+  (symbol (lib_id "Device:C_Polarized") (at 110.49 163.83 0) (unit 1)
+    (in_bom yes) (on_board yes) (dnp no) (fields_autoplaced)
+    (property "Reference" "C2" (at 114.3 162.306 0)
+      (effects (font (size 1.27 1.27)) (justify left))
+    )
+    (property "Value" "100u" (at 114.3 164.846 0)
+      (effects (font (size 1.27 1.27)) (justify left))
+    )
+    (property "Footprint" "Capacitor_THT:CP_Radial_D6.3mm_P2.50mm" (at 111.4552 167.64 0)
+      (effects (font (size 1.27 1.27)) hide)
+    )
+    (property "Datasheet" "~" (at 110.49 163.83 0)
       (effects (font (size 1.27 1.27)) hide)
     )
@@
     )
   )
-  (symbol (lib_id "power:GND") (at 68.58 167.005 0) (unit 1)
-    (in_bom yes) (on_board yes) (dnp no) (fields_autoplaced)
-    (property "Reference" "#PWR04" (at 68.58 173.355 0)
-      (effects (font (size 1.27 1.27)) hide)
-    )
-    (property "Value" "GND" (at 68.58 172.085 0)
-      (effects (font (size 1.27 1.27)))
-    )
-    (property "Footprint" "" (at 68.58 167.005 0)
-      (effects (font (size 1.27 1.27)) hide)
-    )
-    (property "Datasheet" "" (at 68.58 167.005 0)
+  (symbol (lib_id "power:GND") (at 68.58 170.18 0) (unit 1)
+    (in_bom yes) (on_board yes) (dnp no) (fields_autoplaced)
+    (property "Reference" "#PWR04" (at 68.58 176.53 0)
+      (effects (font (size 1.27 1.27)) hide)
+    )
+    (property "Value" "GND" (at 68.58 175.26 0)
+      (effects (font (size 1.27 1.27)))
+    )
+    (property "Footprint" "" (at 68.58 170.18 0)
+      (effects (font (size 1.27 1.27)) hide)
+    )
+    (property "Datasheet" "" (at 68.58 170.18 0)
       (effects (font (size 1.27 1.27)) hide)
     )
@@
   (symbol (lib_id "Connector_Generic:Conn_01x02") (at 237.49 77.47 0) (unit 1)
     (in_bom yes) (on_board yes) (dnp no) (fields_autoplaced)
-    (property "Reference" "J3" (at 240.665 78.105 0)
-      (effects (font (size 1.27 1.27)) (justify left))
-    )
-    (property "Value" "OUTPUT" (at 240.665 80.645 0)
+    (property "Reference" "J3" (at 240.03 78.105 0)
+      (effects (font (size 1.27 1.27)) (justify left))
+    )
+    (property "Value" "Wyjście" (at 240.03 80.645 0)
       (effects (font (size 1.27 1.27)) (justify left))
     )
@@
     )
   )
-  (symbol (lib_id "power:+3V0") (at 110.49 159.385 0) (mirror y) (unit 1)
+  (symbol (lib_id "power:+3V0") (at 110.49 160.02 0) (mirror y) (unit 1)
     (in_bom yes) (on_board yes) (dnp no)
-    (property "Reference" "#PWR013" (at 110.49 163.195 0)
-      (effects (font (size 1.27 1.27)) hide)
-    )
-    (property "Value" "+3V0" (at 110.49 155.575 0)
-      (effects (font (size 1.27 1.27)))
-    )
-    (property "Footprint" "" (at 110.49 159.385 0)
-      (effects (font (size 1.27 1.27)) hide)
-    )
-    (property "Datasheet" "" (at 110.49 159.385 0)
+    (property "Reference" "#PWR013" (at 110.49 163.83 0)
+      (effects (font (size 1.27 1.27)) hide)
+    )
+    (property "Value" "+3V0" (at 110.49 156.21 0)
+      (effects (font (size 1.27 1.27)))
+    )
+    (property "Footprint" "" (at 110.49 160.02 0)
+      (effects (font (size 1.27 1.27)) hide)
+    )
+    (property "Datasheet" "" (at 110.49 160.02 0)
       (effects (font (size 1.27 1.27)) hide)
     )
@@
     )
   )
-  (symbol (lib_id "power:GND") (at 110.49 167.005 0) (unit 1)
-    (in_bom yes) (on_board yes) (dnp no) (fields_autoplaced)
-    (property "Reference" "#PWR014" (at 110.49 173.355 0)
-      (effects (font (size 1.27 1.27)) hide)
-    )
-    (property "Value" "GND" (at 110.49 171.45 0)
-      (effects (font (size 1.27 1.27)))
-    )
-    (property "Footprint" "" (at 110.49 167.005 0)
-      (effects (font (size 1.27 1.27)) hide)
-    )
-    (property "Datasheet" "" (at 110.49 167.005 0)
+  (symbol (lib_id "power:GND") (at 110.49 167.64 0) (unit 1)
+    (in_bom yes) (on_board yes) (dnp no) (fields_autoplaced)
+    (property "Reference" "#PWR014" (at 110.49 173.99 0)
+      (effects (font (size 1.27 1.27)) hide)
+    )
+    (property "Value" "GND" (at 110.49 172.085 0)
+      (effects (font (size 1.27 1.27)))
+    )
+    (property "Footprint" "" (at 110.49 167.64 0)
+      (effects (font (size 1.27 1.27)) hide)
+    )
+    (property "Datasheet" "" (at 110.49 167.64 0)
       (effects (font (size 1.27 1.27)) hide)
     )
@@
   (symbol (lib_id "Connector_Generic:Conn_01x02") (at 63.5 164.465 0) (mirror y) (unit 1)
     (in_bom yes) (on_board yes) (dnp no) (fields_autoplaced)
-    (property "Reference" "J1" (at 63.5 159.385 0)
-      (effects (font (size 1.27 1.27)))
-    )
-    (property "Value" "POWER" (at 63.5 161.925 0)
+    (property "Reference" "J1" (at 63.5 158.75 0)
+      (effects (font (size 1.27 1.27)))
+    )
+    (property "Value" "Zasilanie" (at 63.5 161.29 0)
       (effects (font (size 1.27 1.27)))
     )
@@
     (stroke (width 0.1524) (type solid))
     (fill (color 0 0 0 0.0000))
-    (property "Sheetname" "Autogain" (at 177.165 90.7284 0)
+    (property "Sheetname" "Kontrola Amplitiudy" (at 177.165 90.7284 0)
       (effects (font (size 1.27 1.27)) (justify left bottom))
     )
@@
     (stroke (width 0.1524) (type solid))
     (fill (color 0 0 0 0.0000))
-    (property "Sheetname" "Output Filter" (at 177.8 67.2334 0)
+    (property "Sheetname" "Filtr Wyjściowy" (at 177.8 67.2334 0)
       (effects (font (size 1.27 1.27)) (justify left bottom))
     )
