File: board/weit_generator/weit_generator.kicad_sch (KiCad schematic)
At the start: 19 parts, among them J1 Zasilanie, J2 PROG, J3 Wyjście, U1 AVR32DA28x-xSO, U2 MCP6004, X1 SG-5032CAN

Commit message: Final revision - submitting
Other:
- note added: "Układ napięcia odniesienia"
- moved on the sheet: C10, D1, J3, R20, R23, U?
