File: board/weit_generator/dac.kicad_sch (KiCad schematic)
At the start: 16 parts

Commit message: New layout
Parts:
- renumbered R9 to R10, R10 to R11, R11 to R12, R12 to R13, R13 to R14, R14 to R15, R15 to R16, R16 to R17, R17 to R18, R18 to R19, R3 to R4, R4 to R5, R5 to R6, R6 to R7, R7 to R8, R8 to R9

Commit message: .
Parts:
- renumbered R10 to R1, R7 to R10, R4 to R11, R13 to R12, R14 to R13, R12 to R14, R6 to R16, R5 to R18, R17 to R2, R11 to R3, R19 to R4, R16 to R5, R9 to R6, R15 to R7, R18 to R8, R8 to R9

Commit message: .
Other:
- note added: "R-2R 8-bit volatage-mode DAC. 0.1% or better resistors are highly recommended."
- note removed: "R-2R 8-bit volatage-mode DAC. 1% or better resistors are highly recommended. By Thévenin's theorem Output impedance is 1k"
Changed lines of the file:
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@@
     (effects (font (size 1.27 1.27)) (justify left bottom))
   )
-  (text "R-2R 8-bit volatage-mode DAC. 1% or better resistors are highly recommended.\nBy Thévenin's theorem Output impedance is 1k"
+  (text "R-2R 8-bit volatage-mode DAC. 0.1% or better resistors are highly recommended."
     (at 179.07 171.45 0)
     (effects (font (size 1.27 1.27)) (justify left bottom))

Commit message: WIELKA POLONIAAAAA
Other:
- note removed: "DAC"
- note removed: "R-2R 8-bit volatage-mode DAC. 0.1% or better resistors are highly recommended."
- title: (none) -> Przetwornik Cyfrowo-Analogowy
Changed lines of the file:
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@@
 (kicad_sch (version 20230121) (generator eeschema)
   (paper "A4")
+  (title_block
+    (title "Przetwornik Cyfrowo-Analogowy")
+    (date "2023-04-15")
+    (rev "1.0")
+    (comment 2 "8-biowy napięciowy konwerter R-2R. Rezystory 0.1% lub lepsze")
+  )
   (junction (at 152.4 62.23) (diameter 0) (color 0 0 0 0)
   )
@@
     (stroke (width 0) (type default))
   )
-  (text "DAC" (at 186.055 190.5 0)
-    (effects (font (size 1.27 1.27)) (justify left bottom))
-  )
-  (text "R-2R 8-bit volatage-mode DAC. 0.1% or better resistors are highly recommended."
-    (at 179.07 171.45 0)
-    (effects (font (size 1.27 1.27)) (justify left bottom))
-  )
   (label "BUS5" (at 144.78 77.47 180) (fields_autoplaced)
